File: UcD.kicad_pcb (KiCad board)
At the start: 2 copper layers, 82 x 75 mm, 63 parts, among them J1 Conn_01x02_Male, J2 Conn_01x02_Male, Q1 BF821, Q10 BC857, Q11 BC857, Q12 BC857, Q13 BC857, Q14 IRF540N, Q15 IRF540N, Q16 PZT2222A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

Commit message: AGP2923 STEP model added
Parts:
- moved L1 51.4 mm to (142.6, 73.4), turned to 90 degrees
Changed lines of the file:
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@@
   )
   (footprint "UcD:Inductor_Coilcraft_AGP2923-103KL-17.0x27.0mm" (layer "F.Cu")
-    (at 193.951822 71.986968)
+    (at 142.584322 73.414468 90)
     (descr "Shielded High Current Power Inductor, Coilcraft, AGP2923-103KL, 17.0mmx27.0mm https://www.coilcraft.com/pdfs/agp2923.pdf")
     (tags "inductor Coilcraft tht")
@@
     (property "Sheetname" "")
     (attr through_hole)
-    (fp_text reference "L1" (at -17.48 -16.25) (layer "F.SilkS")
+    (fp_text reference "L1" (at -17.48 -16.25 90) (layer "F.SilkS")
       (effects (font (size 1 1) (thickness 0.15)))
     )
-    (fp_text value "AGP2923-103KL" (at 0 15.75) (layer "F.Fab")
+    (fp_text value "AGP2923-103KL" (at 0 15.75 90) (layer "F.Fab")
       (effects (font (size 1 1) (thickness 0.15)))
     )
-    (fp_text user "${REFERENCE}" (at 0.74 0.82) (layer "F.Fab")
+    (fp_text user "${REFERENCE}" (at 0.74 0.82 90) (layer "F.Fab")
       (effects (font (size 1 1) (thickness 0.15)))
     )
+    (fp_line (start -19.48 -14.75) (end -18.48 -14.75) (layer "F.SilkS") (width 0.12))
     (fp_line (start -19.48 -14.75) (end -19.48 -11.75) (layer "F.SilkS") (width 0.12))
-    (fp_line (start -19.48 -14.75) (end -18.48 -14.75) (layer "F.SilkS") (width 0.12))
-    (pad "" np_thru_hole circle locked (at -5.695 8.09) (size 2.24 2.24) (drill 2.24) (layers *.Cu *.Mask))
-    (pad "" np_thru_hole circle locked (at 5.685 8.09) (size 2.24 2.24) (drill 2.24) (layers *.Cu *.Mask))
-    (pad "" np_thru_hole circle locked (at 5.685 -7.81) (size 2.24 2.24) (drill 2.24) (layers *.Cu *.Mask))
-    (pad "" np_thru_hole circle locked (at -5.695 -7.81) (size 2.24 2.24) (drill 2.24) (layers *.Cu *.Mask))
-    (pad "1" thru_hole oval locked (at 2.61 -7.81) (size 2.35 5.93) (drill oval 1.75 5.33) (layers *.Cu *.Mask)
+    (pad "" np_thru_hole circle (at 5.685 8.09 90) (size 2.24 2.24) (drill 2.24) (layers *.Cu *.Mask))
+    (pad "" np_thru_hole circle (at -5.695 8.09 90) (size 2.24 2.24) (drill 2.24) (layers *.Cu *.Mask))
+    (pad "" np_thru_hole circle (at -5.695 -7.81 90) (size 2.24 2.24) (drill 2.24) (layers *.Cu *.Mask))
+    (pad "" np_thru_hole circle (at 5.685 -7.81 90) (size 2.24 2.24) (drill 2.24) (layers *.Cu *.Mask))
+    (pad "1" thru_hole oval (at 2.61 -7.81 90) (size 2.35 5.93) (drill oval 1.75 5.33) (layers *.Cu *.Mask)
       (net 25 "Net-(C3-Pad2)") (pinfunction "1") (pintype "passive"))
-    (pad "2" thru_hole oval locked (at -2.62 8.7) (size 2.35 5.93) (drill oval 1.75 5.33) (layers *.Cu *.Mask)
+    (pad "2" thru_hole oval (at -2.62 8.7 90) (size 2.35 5.93) (drill oval 1.75 5.33) (layers *.Cu *.Mask)
       (net 38 "Net-(C11-Pad1)") (pinfunction "2") (pintype "passive"))
-    (model "${KISYS3DMOD}/UcD.3dshapes/Coilcraft-AGP2923.STEP"
+    (model "C:/Users/steen/Documents/KiCad/6.0/3dmodels/Coilcraft.3dshapes/Coilcraft-AGP2923.STEP"
       (offset (xyz 0 0 2.5))
       (scale (xyz 1 1 1))
